File: hardware/RP2040_DevBoard_v2.kicad_sch (KiCad schematic)
At the start: 38 parts, among them J1 Conn_01x16, J2 Conn_01x16, J3 USB_C_Receptacle_USB2.0, SW1 PTS636 SK25, SW2 PTS636 SK25, U1 AP2112K-3.3, U2 RP2040, U3 W25Q64JVSS, Y1 12MHz

Commit message: Add files via upload
Parts:
- C1, C2, C7: Digi-Key PN (none) -> 478-5010-2-ND; Mfg PN (none) -> 0603YC105KAT2A
- C10, C11, C12, C13, C15, C3, C4, C5, C6, C8, C9: Digi-Key PN (none) -> 478-7018-2-ND; Mfg PN (none) -> 06033C104KAT4A
- C14, C18: Digi-Key PN (none) -> 478-10578-2-ND; Mfg PN (none) -> 0805ZC106KAT2A
- C16, C17: Digi-Key PN (none) -> 478-9370-2-ND; Mfg PN (none) -> 06031A8R0D4T2A
- D1, D3: Digi-Key PN (none) -> NSR0320MW2T3GOSTR-ND; Mfg PN (none) -> NSR0320MW2T3G
- D2: Digi-Key PN (none) -> 1568-COM-16347TR-ND; Mfg PN (none) -> COM-16347
- J1, J2: Digi-Key PN (none) -> 2057-PH1-16-UA-ND; Mfg PN (none) -> PH1-16-UA
- J3: Digi-Key PN (none) -> 2073-USB4105-GF-ATR-ND; Mfg PN (none) -> USB4105-GF-A
- R1, R3: Digi-Key PN (none) -> P1.30KHTR-ND; Mfg PN (none) -> ERJ-3EKF1301V
- R2, R4: Digi-Key PN (none) -> P10.0KHTR-ND; Mfg PN (none) -> ERJ-3EKF1002V
- R5, R6: Digi-Key PN (none) -> P5.10KHTR-ND; Mfg PN (none) -> ERJ-3EKF5101V
- R7, R8: Digi-Key PN (none) -> P27.0HTR-ND; Mfg PN (none) -> ERJ-3EKF27R0V
- SW1, SW2: Digi-Key PN (none) -> CKN12322-2-ND; Mfg PN (none) -> PTS636 SK25 SMTR LFS
- U1: Digi-Key PN (none) -> AP2112K-3.3TRG1DITR-ND; Mfg PN (none) -> AP2112K-3.3TRG1
- U2: Digi-Key PN (none) -> 2648-SC0914(13)TR-ND; Mfg PN (none) -> SC0914(13)
- U3: Digi-Key PN (none) -> W25Q64JVSSIQ-ND; Mfg PN (none) -> W25Q64JVSSIQ
- Y1: Digi-Key PN (none) -> 1923-830108206909TR-ND; Mfg PN (none) -> 830108206909
