File: hardware/RP2040_DevBoard_v2.kicad_pcb (KiCad board)
At the start: 2 copper layers, 26.2 x 49.5 mm, 40 parts, among them J1 Conn_01x16, J2 Conn_01x16, J3 USB_C_Receptacle_USB2.0, SW1 PTS636 SK25, SW2 PTS636 SK25, U1 AP2112K-3.3, U2 RP2040, U3 W25Q64JVSS, Y1 12MHz

Commit message: Add files via upload
Parts:
- J1, J2: moved to B.Cu
- turned J1 to 180 degrees
- turned J2 to 180 degrees
Other:
- board text added: "11PWR 12SIG"
- board text added: "BOOT"
- board text added: "RST"
